Commit message: urdf

File: 1R_arm/robot.urdf (robot description, URDF)
Before this commit: robot 1R_arm, 3 links, 2 joints
Links:
- link second_segment: mass 0.38219574126274397097 -> 0.38219574126274391546

File: 2R_arm/robot.urdf (robot description, URDF)
Before this commit: robot 2R_arm, 1 links, 0 joints
Links:
- added link end, mass 1e-9
- added link first_segment, mass 0.24000231709280137049; collision mesh filename=package:///dc08_m01_dummy.stl; collision mesh filename=package:///ecrou_2.5.stl
- added link second_segment, mass 0.38219574126274397097; collision mesh filename=package:///ecrou_6.stl; collision mesh filename=package:///m2.5x12__list_khwhpz53lblddb__12.stl
- link base: mass 0.82889145530511265658 -> 0.20669339694956753717; geometry collision mesh filename=package:///base.stl; collision mesh filename=package:///dc08_m01_dummy.stl
Joints:
- added joint R1: type revolute, parent base, child first_segment, origin xyz=-1.1975535627776246625e-47 -0.025970000000000013907 0.054800000000000001488 rpy=-1.570796326794896558 2.7163241488879535893e-29 0, axis 0 0 1, limit lower=-1.9198621771937625091 upper=1.9198621771937625091 effort=1 velocity=20
- added joint R2: type revolute, parent first_segment, child second_segment, origin xyz=8.6597395920808478571e-18 -0.17999999999999999334 3.4694469519536141888e-18 rpy=7.4941785995996121514e-29 -3.3306690738754745517e-16 8.7418612599071244369e-15, axis 0 0 1, limit lower=-2.6179938779914944114 upper=2.6179938779914944114 effort=1 velocity=20
- added joint end_frame: type fixed, parent second_segment, child end, origin xyz=1.2674677052518072442e-17 -0.17000000000000003997 0.025969999999999996559 rpy=1.5707963267948943376 -1.4791141972825890141e-31 -1.5777218104420211586e-30, axis 0 0 0
